File: SwimmingBotV0.1.kicad_pcb (KiCad board)
At the start: 2 copper layers, 141 parts, among them P10 ANT, P11 DEBUG, P2 ANALOG, P3 CHRG, P4 BATT, P5 DEBUG_JUMPER, P6 FIN1, P7 FIN2, P8 MOT1, P9 MOT2, Q1 Q_NMOS_DGS, Q10 PMV45EN2, Q11 PMV45EN2, Q12 PMV45EN2, Q13 PMV45EN2, Q14 PMV45EN2, Q15 PMV45EN2, Q2 Q_PMOS_DGS, Q3 Q_NMOS_DGS, Q4 PMV45EN2, Q5 PMV45EN2, Q6 PMV45EN2, Q7 PMV45EN2, Q8 PMV45EN2, Q9 PMV45EN2, U1 LT3470A, U10 TPS6216X, U2 MCP73834, U3 A4960, U4 A4960, U5 HUM-900-PRO, U6 MPU-9250, U8 MAX6034_25, U9 STM32F446-144, X1 CRYSTAL_SMD, Y1 Crystal

Commit message: pcb going, I think done with memory chips
Parts:
- moved C8 9.21 mm to (159.5, 121.5)
- moved C41 3.69 mm to (177.9, 126.5)
- moved C39 1.10 mm to (177.9, 128.0)
- moved C16 0.99 mm to (177.9, 125.0), turned to 180 degrees
Routing:
- net /Digital/CLK_RAM: track 0.00 -> 54.9 mm, vias 0 -> 3
- net /Micro/FMC_NWAIT: track 0.00 -> 50.7 mm, vias 0 -> 3
- net /Micro/FMC_SDNRAS: track 2.06 -> 45.9 mm, vias 1 -> 5
- net /Micro/FMC_NWE: track 0.00 -> 43.0 mm, vias 0 -> 3
- net /Micro/PA12: track 0.00 -> 41.1 mm, vias 0 -> 3
- net /Digital/BL1#: track 0.00 -> 39.6 mm, vias 0 -> 5
- net /Digital/A12: track 32.6 -> 66.4 mm, vias 0 -> 1
- net /Digital/A15: track 50.0 -> 81.8 mm, vias 2 -> 3
- net /Digital/A14: track 50.2 -> 81.3 mm, vias 2 -> 3
- net /Digital/A13: track 0.00 -> 28.6 mm, vias 0 -> 1
- net /Digital/CAS#: track 1.43 -> 28.2 mm, vias 1 -> 3
- net /Digital/BL0#: track 1.70 -> 23.6 mm, vias 1 -> 3
- net /Digital/A17: track 10.7 -> 28.8 mm, vias 2 -> 3
- net /Digital/A18: track 11.4 -> 28.3 mm, vias 2 -> 3
- net GND: track 83.9 -> 95.9 mm, vias 7 -> 8
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
Commit message: hoh, working on power stuffs now
Parts:
- D1, Q1: moved to B.Cu
- moved R11 200.1 mm to (194.6, 41.6)
- moved R10 192.7 mm to (195.4, 47.8)
- moved L2 191.9 mm to (39.4, 133.8)
- moved U10 188.6 mm to (33.8, 133.2)
- moved P10 173.7 mm to (193.2, 153.7)
- moved C18 173.0 mm to (165.3, 36.0)
- moved C19 170.2 mm to (164.8, 39.0)
- moved C26 169.2 mm to (162.5, 38.7)
- moved C25 169.1 mm to (165.3, 40.7)
- moved C20 168.0 mm to (162.6, 40.2)
- moved C21 167.0 mm to (165.2, 43.2)
- moved C24 165.6 mm to (165.0, 44.9)
- moved C23 165.5 mm to (162.2, 42.9)
- moved Q10 164.9 mm to (190.1, 23.7)
- moved Q7 164.9 mm to (190.6, 20.7)
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Connections:
- P4 pad 4: /Charge/2S -> /Charge/2S_RAW
- P5 pad 1: /Charge/2S -> /Charge/2S_RAW
Routing:
- net GND: track 95.9 -> 147.8 mm, vias 8 -> 18
- net /Charge/1S: track 0.00 -> 33.5 mm
- net Net-(C7-Pad1): track 0.00 -> 18.5 mm, vias 0 -> 1
- net /Charge/5V_CHG: track 0.00 -> 17.0 mm
- net /Charge/2S_NEG: track 0.00 -> 15.1 mm
- net /Charge/CHG_STAT2: track 0.00 -> 13.4 mm, vias 0 -> 2
- net /Charge/CHG_STAT1: track 3.75 -> 17.0 mm, vias 0 -> 2
- net /Charge/2S_EN: track 0.00 -> 7.49 mm, vias 0 -> 2
- net /Charge/2S: track 0.00 -> 6.68 mm
- net /Charge/CHG_EN#: track 0.00 -> 5.12 mm, vias 0 -> 1
- net Net-(R2-Pad1): track 0.00 -> 5.03 mm, vias 0 -> 1
- net /Power/CHG_CTL_VCC: track 26.5 -> 31.3 mm
- net Net-(C6-Pad1): track 0.00 -> 4.28 mm
- net /Charge/CHG_TE#: track 0.00 -> 4.04 mm, vias 0 -> 1
- net /Charge/2S_RAW: track 0.00 -> 3.76 mm
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- added copper zone on B.Cu, net /Charge/1S
- added copper zone on F.Cu, net /Charge/1S
- added copper zone on B.Cu, net /Charge/2S
- added copper zone on F.Cu, net /Charge/2S_NEG
- added copper zone on F.Cu, net /Charge/5V_CHG
- added copper zone on B.Cu, net GND
- added copper zone on F.Cu, net GND

Commit message: woohoo getting there
Parts:
- removed W3: GND, Measurement_Points:Measurement_Point_Round-SMD-Pad_Small
- removed W6: VBAT, Measurement_Points:Measurement_Point_Round-SMD-Pad_Small
- removed W7: AUX_3.3V, Measurement_Points:Measurement_Point_Round-SMD-Pad_Small
- C1, C18, C22, C24, C28, C33, C34, C43, C45, C49, C50, C57, C60, C61, C63, C64, C67, C68, D4, D5, JP1, P9, R17, R19, R20, R8, R9, U8: moved to B.Cu
- moved Q13 206.1 mm to (43.8, 161.4), turned to 180 degrees
- moved Q12 199.5 mm to (47.7, 162.6), turned to 180 degrees
- moved Q8 198.5 mm to (54.5, 161.9), turned to 270 degrees
- moved Q14 196.6 mm to (68.0, 168.8), turned to 270 degrees
- moved Q11 195.6 mm to (75.0, 171.8), turned to 270 degrees
- moved Q9 194.8 mm to (51.2, 162.9), turned to 270 degrees
- moved Q5 191.6 mm to (57.8, 161.9), turned to 270 degrees
- moved Q15 191.5 mm to (65.0, 164.2), turned to 270 degrees
- moved Q4 187.5 mm to (58.0, 158.1)
- moved R10 186.7 mm to (41.2, 153.0), turned to 90 degrees
- moved Q7 186.3 mm to (75.0, 166.8), turned to 270 degrees
- moved Q10 184.0 mm to (79.0, 170.2)
- moved P10 178.8 mm to (14.4, 156.2)
- moved U4 178.1 mm to (49.5, 154.0), turned to 270 degrees
- moved Q6 174.6 mm to (79.0, 165.2)
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Connections:
- MEM1 pad 40: (no net) -> Net-(MEM1-Pad40)
- MEM2 pad 16: (no net) -> Net-(MEM2-Pad16)
- MEM2 pad 27: (no net) -> Net-(MEM2-Pad27)
- MEM2 pad 28: (no net) -> Net-(MEM2-Pad28)
- MEM2 pad 30: (no net) -> Net-(MEM2-Pad30)
- MEM2 pad 53: (no net) -> Net-(MEM2-Pad53)
- MEM2 pad 55: (no net) -> Net-(MEM2-Pad55)
- MEM2 pad 56: (no net) -> Net-(MEM2-Pad56)
- P8 pad 1: /Motors/A1 -> /Motors/C1
- P8 pad 3: /Motors/C1 -> /Motors/A1
- P9 pad 1: /Motors/A2 -> /Motors/C2
- P9 pad 3: /Motors/C2 -> /Motors/A2
- R17 pad 2: /Micro/PG11 -> /Micro/PF7
- R20 pad 2: /Micro/PG12 -> /Micro/PF8
- U1 pad 7: (no net) -> Net-(U1-Pad7)
- U1 pad 8: /Micro/PD3 -> /Micro/PG12
- U10 pad 8: (no net) -> /Power/AUX_3.3V_GOOD
- U3 pad PAD: (no net) -> Net-(U3-PadPAD)
- U4 pad PAD: (no net) -> Net-(U4-PadPAD)
- U5 pad 1: (no net) -> Net-(U5-Pad1)
- U5 pad 10: (no net) -> Net-(U5-Pad10)
- U5 pad 11: (no net) -> Net-(U5-Pad11)
- U5 pad 12: /Micro/PC10 -> /Micro/PG7
- U5 pad 13: /Micro/PC5 -> /Micro/PG6
- U5 pad 2: (no net) -> Net-(U5-Pad2)
- U5 pad 23: (no net) -> Net-(U5-Pad23)
- U5 pad 24: (no net) -> Net-(U5-Pad24)
- U5 pad 28: (no net) -> Net-(U5-Pad28)
- U5 pad 3: (no net) -> Net-(U5-Pad3)
- U5 pad 30: (no net) -> Net-(U5-Pad30)
- U5 pad 31: (no net) -> Net-(U5-Pad31)
- U5 pad 32: (no net) -> Net-(U5-Pad32)
- U5 pad 4: (no net) -> Net-(U5-Pad4)
- U5 pad 5: (no net) -> Net-(U5-Pad5)
- U5 pad 6: (no net) -> Net-(U5-Pad6)
- U5 pad 7: /Micro/PC1 -> /Micro/PB14
- U5 pad 8: /Micro/PC4 -> /Micro/PB15
- U6 pad 14: (no net) -> Net-(U6-Pad14)
- U6 pad 15: (no net) -> Net-(U6-Pad15)
- U6 pad 16: (no net) -> Net-(U6-Pad16)
- U6 pad 17: (no net) -> Net-(U6-Pad17)
- U6 pad 19: (no net) -> Net-(U6-Pad19)
- U6 pad 2: (no net) -> Net-(U6-Pad2)
- U6 pad 21: (no net) -> /Sensors/AUX_SDA
- U6 pad 3: (no net) -> Net-(U6-Pad3)
- U6 pad 4: (no net) -> Net-(U6-Pad4)
- U6 pad 5: (no net) -> Net-(U6-Pad5)
- U6 pad 6: (no net) -> Net-(U6-Pad6)
- U6 pad 7: (no net) -> /Sensors/AUX_SCL
- U9 pad 111: /Micro/PC10 -> /Charge/CHG_TE#
- U9 pad 112: (no net) -> /Micro/DCMI_D4
- U9 pad 113: /Sensors/GYRO_INT -> /Charge/2S_EN
- U9 pad 116: (no net) -> /Micro/SDIO_CMD
- U9 pad 117: /Micro/PD3 -> /Micro/DCMI_D5
- U9 pad 124: (no net) -> /Micro/DCMI_VSYNC
- U9 pad 125: (no net) -> /Micro/DCMI_D2
- U9 pad 126: /Micro/PG11 -> /Charge/CHG_STAT2
- U9 pad 136: (no net) -> /Micro/SCL
- U9 pad 137: /Charge/CHG_STAT2 -> /Micro/SDA
- U9 pad 139: (no net) -> /Micro/DCMI_D6
- U9 pad 140: (no net) -> /Micro/DCMI_D7
- U9 pad 18: /Motors/MOT1_CS# -> /Sensors/GYRO_INT
- U9 pad 19: /Motors/MOT2_CS# -> /Micro/PF7
- U9 pad 20: /Motors/MOT1_RESET# -> /Micro/PF8
- U9 pad 21: /Motors/MOT2_RESET# -> /Micro/PF9
- U9 pad 22: /Motors/MOT1_DIAG -> /Micro/PF10
- U9 pad 27: /Micro/PC1 -> /Motors/MOT1_RESET#
- U9 pad 40: (no net) -> /Micro/DCMI_HSYNC
- U9 pad 42: (no net) -> /Micro/DCMI_PIXCLK
- U9 pad 44: /Micro/PC4 -> /Motors/MOT2_DIAG
- U9 pad 45: /Micro/PC5 -> /Motors/MOT2_RESET#
- U9 pad 46: /Charge/CHG_STAT1 -> /Motors/MOT2_CS#
- U9 pad 69: /Micro/SCL -> /Motors/MOT1_CS#
- U9 pad 70: /Micro/SDA -> /Motors/MOT1_DIAG
- U9 pad 73: /Charge/CHG_TE# -> /Charge/CHG_EN#
- U9 pad 74: /Charge/CHG_EN# -> /Charge/CHG_STAT1
- U9 pad 75: /Charge/2S_EN -> /Micro/PB14
- U9 pad 76: /Motors/MOT2_DIAG -> /Micro/PB15
- U9 pad 91: (no net) -> /Micro/PG6
- U9 pad 92: (no net) -> /Micro/PG7
- U9 pad 96: (no net) -> /Micro/DCMI_D0
- U9 pad 97: (no net) -> /Micro/DCMI_D1
- U9 pad 98: (no net) -> /Micro/SDIO_D0
- U9 pad 99: (no net) -> /Micro/DCMI_D3
Routing:
- net GND: track 147.8 -> 432.1 mm, vias 18 -> 54
- net /Charge/2S: track 6.68 -> 133.7 mm, vias 0 -> 7
- net /Motors/MOT2_TACH: track 0.00 -> 111.8 mm, vias 0 -> 6
- net /Motors/SDO: track 0.00 -> 111.4 mm, vias 0 -> 6
- net /Power/CHG_CTL_VCC: track 31.3 -> 131.9 mm, vias 2 -> 15
- net /Digital/3.3V: track 63.0 -> 142.9 mm, vias 10 -> 17
- net /Micro/MOT1_PWM: track 0.00 -> 79.8 mm, vias 0 -> 4
- net /Charge/5V_CHG: track 17.0 -> 78.6 mm
- net /Motors/FIN1: track 0.00 -> 58.6 mm, vias 0 -> 1
- net /Motors/LSS2: track 0.00 -> 58.3 mm, vias 0 -> 5
- net /Charge/CHG_STAT2: track 13.4 -> 69.5 mm, vias 2 -> 6
- net /Motors/C1: track 0.00 -> 55.3 mm, vias 0 -> 3
- net /Motors/SCK: track 0.00 -> 54.1 mm, vias 0 -> 4
- net /Motors/SDI: track 2.82 -> 54.7 mm, vias 0 -> 4
- net /Motors/MOT1_TACH: track 0.00 -> 51.5 mm, vias 0 -> 2
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- added copper zone on F.Cu, net /Charge/2S
- added copper zone on F.Cu, net /Digital/3.3V
- added copper zone on F.Cu, net /Motors/LSS
- added copper zone on F.Cu, net /Motors/LSS2
- added copper zone on F.Cu, net /Power/CHG_CTL_VCC
- added copper zone on F.Cu, net Net-(C40-Pad1)
- added copper zone on F.Cu, net Net-(L2-Pad2)
Other:
- board outline added: 70 x 51 mm

Commit message: done with connections, just needs plane cleanup
Parts:
- removed C36, C48: 100nF, Capacitors_SMD:C_0402
- added REF**: MountingHole_2.2mm_M2, Mounting_Holes:MountingHole_2.2mm_M2, F.Cu at (15.0, 150.0)
- moved W1 32.4 mm to (72.3, 194.5)
- moved W2 28.2 mm to (70.3, 194.5)
- moved C54 27.8 mm to (31.9, 182.9), turned to 90 degrees
- moved C42 1.25 mm to (29.9, 177.6)
- moved P10 1.21 mm to (14.4, 155.0)
- moved C55 1.17 mm to (31.9, 186.7)
- moved C40 1.05 mm to (30.5, 179.3), turned to 180 degrees
- moved C53 0.65 mm to (31.9, 191.7)
- moved R13 0.57 mm to (62.0, 196.3), turned to 270 degrees
- moved R16 0.53 mm to (25.9, 182.2)
- moved C9 0.09 mm to (43.2, 185.1)
Routing:
- net GND: track 432.1 -> 630.8 mm, vias 54 -> 79
- net /Digital/3.3V: track 142.9 -> 306.2 mm, vias 17 -> 29
- net /Charge/2S: track 133.7 -> 266.9 mm, vias 7 -> 17
- net /Power/CHG_CTL_VCC: track 131.9 -> 264.8 mm, vias 15 -> 27
- net /Micro/PG6: track 2.22 -> 72.1 mm, vias 0 -> 2
- net /Micro/PB15: track 0.00 -> 48.0 mm, vias 0 -> 2
- net /Micro/PB14: track 0.00 -> 44.5 mm, vias 0 -> 2
- net /Micro/PG7: track 26.7 -> 61.5 mm, vias 3 -> 4
- net /Motors/LSS: track 44.3 -> 53.8 mm
- net /Micro/RST#: track 36.8 -> 45.5 mm
- net /Micro/FMC_NWE: track 43.0 -> 48.8 mm
- net Net-(P10-Pad1): track 0.00 -> 5.70 mm
- net /Micro/PA12: track 41.1 -> 45.3 mm
- net /Micro/FMC_NWAIT: track 53.6 -> 57.4 mm
- net /Digital/DQ8: track 49.7 -> 46.0 mm
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
Commit message: PCB layout rev 1 done
Routing:
- net /Charge/2S: track 266.9 -> 280.5 mm, vias 17 -> 23
- net /Digital/3.3V: track 306.2 -> 310.0 mm
- net /Digital/A0: track 27.0 -> 29.5 mm
- net /Power/CHG_CTL_VCC: track 264.8 -> 266.3 mm
- net /Micro/A2: track 37.1 -> 35.8 mm
- net /Motors/B2: track 27.9 -> 26.7 mm
- net /Digital/A17: track 29.8 -> 30.7 mm
- net /Digital/DQ6: track 90.2 -> 91.0 mm
- net GND: track 630.8 -> 630.1 mm
- net /Digital/DQ4: track 91.4 -> 92.0 mm
- net /Digital/DQ5: track 92.5 -> 93.1 mm
