File: SwimminBotV0.1-rf.sch (KiCad schematic (older format))
At the start: 4 parts, among them P10 ANT, U5 HUM-900-PRO

Commit message: swapped out battery serializing hardware from discrete to IC, and standard level fets
Connections:
- net RF_CTS: now reaches U5.28 (CTS#)
- net RF_ACTV: now reaches U5.30 (RFACTV)
- net RF_TXE: now reaches U5.31 (BE)
- no-connect marks 5 -> 2
Changed lines of the file:
@@
 Text Label 3750 3000 0    60   ~ 0
 GND
-NoConn ~ 3350 2500
-NoConn ~ 3250 2500
 Text Notes 2950 1800 0    60   ~ 0
 call it 50mA
-NoConn ~ 3750 3100
 Wire Wire Line
 	3750 3700 3850 3700
@@
 Text Label 2000 5300 0    60   ~ 0
 GND
+Text HLabel 3800 3100 2    60   Input ~ 0
+RF_CTS
+Wire Wire Line
+	3750 3100 3800 3100
+Text HLabel 3350 2450 1    60   Input ~ 0
+RF_ACTV
+Wire Wire Line
+	3350 2500 3350 2450
+Text HLabel 3250 2450 1    60   Input ~ 0
+RF_TXE
+Wire Wire Line
+	3250 2500 3250 2450
 $EndSCHEMATC
