File: SwimmingBotV0.1.sch (KiCad schematic (older format))
At the start: 14 parts, among them P1 DCMI, P2 ANALOG, P5 CONN_01X08

Commit message: submitted to fab woohoo
Parts:
- P5: value CONN_01X08 -> GPIO
Connections:
- net GND: now also P2.1 (P1); no longer P2.4 (P4)
- net Micro/A1: now also P2.4 (P4); no longer P2.1 (P1)
- net Micro/A2: now also P2.3 (P3); no longer P2.2 (P2)
- net Micro/A3: now also P2.2 (P2); no longer P2.3 (P3)
Changed lines of the file:
@@
 F 3 "" H 6800 7400 50  0000 C CNN
 	1    6800 7400
-	1    0    0    -1
+	1    0    0    1
 $EndComp
 Text Label 6550 7150 0    60   ~ 0
@@
 P 9750 3600
 F 0 "P5" H 9750 4050 50  0000 C CNN
-F 1 "CONN_01X08" V 9850 3600 50  0000 C CNN
+F 1 "GPIO" V 9850 3600 50  0000 C CNN
 F 2 "Pin_Headers:Pin_Header_Straight_2x04_Pitch1.27mm" H 9750 3600 50  0001 C CNN
 F 3 "" H 9750 3600 50  0000 C CNN
